Commit message: add mithmd

File: legged_examples/legged_bipedv5_description/urdf/bipedv5_sim.urdf (robot description, URDF)
Before this commit: robot bipedv5, 18 links, 17 joints
Joints:
- joint lap: limit lower=-0.15 upper=0.15 effort=100 velocity=100 -> lower=-0.2 upper=0.2 effort=100 velocity=100
- joint lkp: axis 1 0 0 -> (none); limit lower=-0.15 upper=0.15 effort=100 velocity=100 -> (none); type prismatic -> fixed
- joint rap: limit lower=-0.1 upper=0.1 effort=100 velocity=100 -> lower=-0.2 upper=0.2 effort=100 velocity=100
- joint rkp: axis 1 0 0 -> (none); limit lower=-0.1 upper=0.1 effort=100 velocity=100 -> (none); type prismatic -> fixed
