Commit message: a

File: legged_examples/legged_bipedv5_description/urdf/bipedv5.urdf (robot description, URDF)
Before this commit: robot bipedv5, 18 links, 17 joints
Links:
- link left_ankle_Link: geometry collision box size=0.12 0.22 0.01; visual mesh filename=package://legged_bipedv5_description/meshes/left_ankle_Link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
- link right_ankle_Link: geometry collision box size=0.12 0.22 0.01; visual mesh filename=package://legged_bipedv5_description/meshes/right_ankle_Lin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
